File: NMEA_Multiplexer_v2.sch (KiCad schematic (older format))
At the start: 31 parts

Commit message: First complete schematic
Parts:
- removed C? (x9): 100n, symbol C_Small
- removed C? (x2): 4.7u, symbol C_Small
- removed C?: 2.2u, symbol C_Small
- removed D? (x7): LED_Dual_ACA, symbol LED_Dual_ACA
- added C1, C11: 4.7u, Capacitors_SMD:C_0603, symbol C_Small
- added C10, C12, C14, C16, C17, C18, C19, C2, C20, C21, C22, C23, C24, C25, C26, C27, C29, C3, C4, C5, C6, C7, C8: 100n, Capacitors_SMD:C_0603, symbol C_Small
- added C28: 10u, Capacitors_SMD:CP_Elec_4x5.8, symbol CP_Small
- added C9: 2.2u, Capacitors_SMD:C_0603, symbol C_Small
- added D1: Rx 0 (green), LEDs:LED_0603, symbol LED
- added D10: Rx 3 (green), LEDs:LED_0603, symbol LED
- added D11: Tx 3 (green), LEDs:LED_0603, symbol LED
- added D12: Err 3 (red), LEDs:LED_0603, symbol LED
- added D13: Rx 4 (green), LEDs:LED_0603, symbol LED
- added D14: Tx 4 (green), LEDs:LED_0603, symbol LED
- added D15: Err 4 (red), LEDs:LED_0603, symbol LED
- added D16: Rx BT (green), LEDs:LED_0603, symbol LED
- added D17: Tx BT (green), LEDs:LED_0603, symbol LED
- added D18: Err BT (red), LEDs:LED_0603, symbol LED
- added D19: BT Con (blue), LEDs:LED_0603, symbol LED
- added D2: Tx 0 (green), LEDs:LED_0603, symbol LED
- added D20: USB Con (green), LEDs:LED_0603, symbol LED
- added D21: PWR (green), LEDs:LED_0603, symbol LED
- added D3: Err 0 (red), LEDs:LED_0603, symbol LED
- added D4: Rx 1 (green), LEDs:LED_0603, symbol LED
- added D5: Tx 1 (green), LEDs:LED_0603, symbol LED
- added D6: Err 1 (red), LEDs:LED_0603, symbol LED
- added D7: Rx 2 (green), LEDs:LED_0603, symbol LED
- added D8: Tx (green), LEDs:LED_0603, symbol LED
- added D9: Err 2 (red), LEDs:LED_0603, symbol LED
- added J2: Port 1, Connectors_Terminal_Blocks:TerminalBlock_Pheonix_PT-3.5mm_3pol, symbol Screw_Terminal_1x03
- added J3: Port 2, Connectors_Terminal_Blocks:TerminalBlock_Pheonix_PT-3.5mm_3pol, symbol Screw_Terminal_1x03
- added J4: Port 3, Connectors_Terminal_Blocks:TerminalBlock_Pheonix_PT-3.5mm_3pol, symbol Screw_Terminal_1x03
- added J5: Port 4, Connectors_Terminal_Blocks:TerminalBlock_Pheonix_PT-3.5mm_3pol, symbol Screw_Terminal_1x03
- added J6: Port 5, Connectors_Terminal_Blocks:TerminalBlock_Pheonix_PT-3.5mm_3pol, symbol Screw_Terminal_1x03
- added J7: 12V, Connectors_Terminal_Blocks:TerminalBlock_Pheonix_PT-3.5mm_2pol, symbol Screw_Terminal_1x02
- added J8: DEBUG UART, Pin_Headers:Pin_Header_Straight_1x03_Pitch2.54mm, symbol CONN_01X03
- added R1, R10, R11, R12, R13, R14, R15, R16, R17, R18, R19, R2, R20, R21, R3, R4, R5, R6, R7, R8, R9: 220, Resistors_SMD:R_0603, symbol R
- added R24: 27k, Resistors_SMD:R_0603, symbol R
- added R25: 47k, Resistors_SMD:R_0603, symbol R
- added R29, R31: 39, Resistors_SMD:R_0603, symbol R
- added R30: 100k, Resistors_SMD:R_0603, symbol R
- added SW1: Reset, Buttons_Switches_SMD:SW_SPST_EVQP2, symbol SW_Push
- added U2, U3: XR32330, Housings_DFN_QFN:QFN-24_4x4mm_Pitch0.5mm_NoMask, symbol XR32330
- added U4: LF33ABDT-TR, TO_SOT_Packages_SMD:TO-252-2_Rectifier, symbol LF33ABDT-TR
- added U5: HM-11, MaxNil:HM-11, symbol HM-11-RESCUE-NMEA_Multiplexer_v2
- C13, C15: renamed from C?; footprint (none) -> Capacitors_SMD:C_0603
- J1: renamed from J?; footprint (none) -> Connectors:USB_Mini-B
- J9: renamed from J?; footprint (none) -> Pin_Headers:Pin_Header_Straight_2x05_Pitch1.27mm_SMD
- JP1: renamed from JP?; footprint (none) -> Resistors_SMD:R_0603
- R22, R23, R26, R27, R28: renamed from R?; footprint (none) -> Resistors_SMD:R_0603
- U1: renamed from U?; footprint LQFP64 -> Housings_QFP:LQFP-64_10x10mm_Pitch0.5mm
- Y1: renamed from Y?; footprint (none) -> Crystals:Crystal_SMD_3215-2pin_3.2x1.5mm
Connections:
- net labels added: BT_RESET_N, CTS7, LED_0_ERR, LED_0_RX, LED_0_TX, LED_1_ERR, LED_1_RX, LED_1_TX, LED_2_ERR, LED_2_RX, LED_2_TX, LED_3_ERR, LED_3_RX, LED_3_TX, LED_4_ERR, LED_4_RX, LED_4_TX, LED_BT_CON, LED_BT_ERR, LED_BT_RX, LED_BT_TX, LED_USB_CON, RTS7, RX0, RX1, RX2, RX3, RX4, TX0, TX1, TX2, TX3, TX4, VBUS_3.3V
- net labels removed: RXD6, TXD6, VBUS
- wire segments 117 -> 348
- no-connect marks 3 -> 19
Other:
- note added: "Close to\nVDDCORE"
- note added: "Close to\nVDDIO"
- note added: "Close to\nVDDOUT"
- note added: "Close to\nVDDUSB"
- note removed: "Close to VDDCORE"
- note removed: "Close to VDDIO"
- note removed: "Close to VDDOUT"
- note removed: "Close to VDDUSB"

Commit message: Fixed some pin-errors in the ATSAM symbol Swapped place between LED and resistor
Connections:
- wire segments 348 -> 404

Commit message: Schematic ok Most of components placed on PCB
Parts:
- removed D18: Err BT (red), LEDs:LED_0603, symbol LED
- removed R18: 220, Resistors_SMD:R_0603, symbol R
- JP1: footprint Resistors_SMD:R_0603 -> Pin_Headers:Pin_Header_Straight_1x02_Pitch2.54mm
Connections:
- wire segments 404 -> 339

Commit message: Before the renaming
Connections:
- net labels removed: LED_BT_ERR
- wire segments 339 -> 338
- no-connect marks 19 -> 20
Changed lines of the file:
@@
 RXD7
 Text Label 4900 2850 2    60   ~ 0
-TXD4
+TXD5
 Text Label 4900 2950 2    60   ~ 0
-RXD4
+RXD5
 Text Label 9100 2150 0    60   ~ 0
 TXD3
@@
 RXD3
 Text Label 9100 2350 0    60   ~ 0
+RXD4
+Text Label 9100 2450 0    60   ~ 0
+TXD4
+Text Label 9100 2750 0    60   ~ 0
 RXD2
-Text Label 9100 2450 0    60   ~ 0
+Text Label 9100 2850 0    60   ~ 0
 TXD2
-Text Label 9100 2750 0    60   ~ 0
-RXD0
-Text Label 9100 2850 0    60   ~ 0
-TXD0
 Text Label 9100 3050 0    60   ~ 0
-RXD5
+RXD1
 Text Label 9100 3150 0    60   ~ 0
-TXD5
+TXD1
 Text Label 9100 2950 0    60   ~ 0
 LED_3_TX
@@
 LED_3_ERR
 Text Label 4900 2250 2    60   ~ 0
-RXD1
+RXD0
 Text Label 4900 2350 2    60   ~ 0
-TXD1
+TXD0
 Text Label 9100 3950 0    60   ~ 0
 DM
@@
 Text Label 4900 3150 2    60   ~ 0
 LED_BT_TX
-Text Label 4900 3350 2    60   ~ 0
-LED_BT_ERR
 Text Label 4900 3550 2    60   ~ 0
 LED_USB_CON
@@
 	9100 3450 9000 3450
 Wire Wire Line
-	4900 3350 5000 3350
-Wire Wire Line
 	4900 3550 5000 3550
 Wire Wire Line
@@
 	3550 1300 3300 1300
 Text Label 3550 900  0    60   ~ 0
-TX0
+TX2
 Text Label 3550 1300 0    60   ~ 0
-RX0
+RX2
 $Comp
 L GND #PWR045
@@
 	3550 3300 3300 3300
 Text Label 3550 2900 0    60   ~ 0
-TX2
+TX0
 Text Label 3550 3300 0    60   ~ 0
-RX2
+RX0
 $Comp
 L GND #PWR047
@@
 	1    0    0    -1
 $EndComp
+NoConn ~ 5000 3350
 $EndSCHEMATC

Commit message: Fixed missing decaps on VDDCORE
Parts:
- removed D20: USB Con (green), LEDs:LED_0603, symbol LED
- removed R20: 220, Resistors_SMD:R_0603, symbol R
Connections:
- net labels added: +1V8, CTS0, RTS0, RXD6, TXD6
- net labels removed: CTS7, LED_USB_CON, RTS7, RXD7, TXD7
- wire segments 338 -> 394
- no-connect marks 20 -> 22

Commit message: Swapped LED_BT_TX with LED_BT_RX
Parts:
- D1: renamed from D11; value Tx 3 (green) -> Tx 3 (gReen)
- D11: renamed from D8; value Tx (green) -> Tx (gReen)
- D12: renamed from D9; value Err 2 (red) -> ERr 2 (reD)
- D14: renamed from D5; value Tx 1 (green) -> Tx 1 (gReen)
- D15: renamed from D6; value Err 1 (red) -> ERr 1 (reD)
- D17: renamed from D2; value Tx 0 (green) -> Tx 0 (gReen)
- D18: renamed from D3; value Err 0 (red) -> ERr 0 (reD)
- D2: renamed from D12; value Err 3 (red) -> ERr 3 (reD)
- D4: renamed from D14; value Tx 4 (green) -> Tx 4 (gReen)
- D5: renamed from D15; value Err 4 (red) -> ERr 4 (reD)
- D8: renamed from D19; value BT Con (blue) -> BT Cxon (blue)
- D9: renamed from D17; value Tx BT (green) -> Tx BT (gReen)
- J2: value Port 1 -> PoRt 1
- J3: value Port 2 -> PoRt 2
- J4: value Port 3 -> PoRt 3
- J5: value Port 4 -> PoRt 4
- J6: value Port 5 -> PoRt 5
- JP1: footprint Pin_Headers:Pin_Header_Straight_1x02_Pitch2.54mm -> Pin_Headers:Pin_Header_Straight_1x02_Pitch2.00mm
- renumbered C21 to C1, C3 to C10, C2 to C11, C1 to C12, C29 to C13, C28 to C14, C14 to C15, C20 to C16, C22 to C17, C24 to C18, C17 to C19, C23 to C2, C25 to C20, C16 to C21, C6 to C22, C11 to C23, C12 to C24, C9 to C25, C10 to C26, C4 to C27, C5 to C28, C7 to C29, C26 to C3, C19 to C4, C27 to C5, C18 to C6, C15 to C7, C13 to C8, C8 to C9, D16 to D10, D7 to D13, D4 to D16, D1 to D19, D10 to D3, D13 to D6, D21 to D7, R14 to R1, R19 to R10, R24 to R11, R25 to R12, R11 to R13, R12 to R14, R10 to R15, R22 to R16, R23 to R17, R8 to R18, R7 to R19, R15 to R2, R9 to R20, R4 to R21, R6 to R22, R5 to R23, R26 to R24, R27 to R25, R28 to R26, R1 to R27, R2 to R28, R3 to R29, R13 to R3, R16 to R4, R17 to R5, R21 to R6, R31 to R7, R30 to R8, R29 to R9, U3 to U2, U2 to U3
Connections:
- net labels added: CxTS0, LED_BT_CxON, TCxK
- net labels removed: CTS0, LED_BT_CON, TCK
- wire segments 394 -> 331
- no-connect marks 22 -> 21
Other:
- note added: "Cxlose to\nVDDCORE"
- note added: "Cxlose to\nVDDIO"
- note added: "Cxlose to\nVDDOUT"
- note added: "Cxlose to\nVDDUSB"
- note removed: "Close to\nVDDCORE"
- note removed: "Close to\nVDDIO"
- note removed: "Close to\nVDDOUT"
- note removed: "Close to\nVDDUSB"

Commit message: Swapped values between C11 and C12
Parts:
- C11: value 100n -> 4.7u
- C12: value 4.7u -> 100n
Changed lines of the file:
@@
 P 750 10400
 F 0 "C12" H 760 10470 50  0000 L CNN
-F 1 "4.7u" H 760 10320 50  0000 L CNN
+F 1 "100n" H 760 10320 50  0000 L CNN
 F 2 "Capacitors_SMD:C_0603" H 750 10400 50  0001 C CNN
 F 3 "" H 750 10400 50  0001 C CNN
@@
 P 1000 10400
 F 0 "C11" H 1010 10470 50  0000 L CNN
-F 1 "100n" H 1010 10320 50  0000 L CNN
+F 1 "4.7u" H 1010 10320 50  0000 L CNN
 F 2 "Capacitors_SMD:C_0603" H 1000 10400 50  0001 C CNN
 F 3 "" H 1000 10400 50  0001 C CNN

Commit message: Soon complete
Parts:
- renumbered R15 to R1, R7 to R10, R8 to R11, R9 to R12, R10 to R13, R11 to R14, R12 to R15, R14 to R2, R13 to R3, R1 to R4, R3 to R5, R2 to R6, R4 to R7, R5 to R8, R6 to R9
Changed lines of the file:
@@
 EESchema Schematic File Version 2
-LIBS:NMEA_Multiplexer_v2-rescue
 LIBS:MaxNil_components
 LIBS:74xgxx
@@
 $EndComp
 $Comp
-L R R15
+L R R1
 U 1 1 58F58A63
 P 1900 3750
-F 0 "R15" V 1980 3750 50  0000 C CNN
+F 0 "R1" V 1980 3750 50  0000 C CNN
 F 1 "220" V 1900 3750 50  0000 C CNN
 F 2 "Resistors_SMD:R_0603" V 1830 3750 50  0001 C CNN
@@
 $EndComp
 $Comp
-L R R13
+L R R3
 U 1 1 58F58A69
 P 1900 4050
-F 0 "R13" V 1980 4050 50  0000 C CNN
+F 0 "R3" V 1980 4050 50  0000 C CNN
 F 1 "220" V 1900 4050 50  0000 C CNN
 F 2 "Resistors_SMD:R_0603" V 1830 4050 50  0001 C CNN
@@
 $EndComp
 $Comp
-L R R14
+L R R2
 U 1 1 58F58A6F
 P 1900 4350
-F 0 "R14" V 1980 4350 50  0000 C CNN
+F 0 "R2" V 1980 4350 50  0000 C CNN
 F 1 "220" V 1900 4350 50  0000 C CNN
 F 2 "Resistors_SMD:R_0603" V 1830 4350 50  0001 C CNN
@@
 $EndComp
 $Comp
-L R R3
+L R R5
 U 1 1 58F58EE2
 P 1900 4700
-F 0 "R3" V 1980 4700 50  0000 C CNN
+F 0 "R5" V 1980 4700 50  0000 C CNN
 F 1 "220" V 1900 4700 50  0000 C CNN
 F 2 "Resistors_SMD:R_0603" V 1830 4700 50  0001 C CNN
@@
 $EndComp
 $Comp
-L R R1
+L R R4
 U 1 1 58F58EE8
 P 1900 5000
-F 0 "R1" V 1980 5000 50  0000 C CNN
+F 0 "R4" V 1980 5000 50  0000 C CNN
 F 1 "220" V 1900 5000 50  0000 C CNN
 F 2 "Resistors_SMD:R_0603" V 1830 5000 50  0001 C CNN
@@
 $EndComp
 $Comp
-L R R2
+L R R6
 U 1 1 58F58EEE
 P 1900 5300
-F 0 "R2" V 1980 5300 50  0000 C CNN
+F 0 "R6" V 1980 5300 50  0000 C CNN
 F 1 "220" V 1900 5300 50  0000 C CNN
 F 2 "Resistors_SMD:R_0603" V 1830 5300 50  0001 C CNN
@@
 $EndComp
 $Comp
-L R R4
+L R R7
 U 1 1 58F58F1D
 P 1900 5700
-F 0 "R4" V 1980 5700 50  0000 C CNN
+F 0 "R7" V 1980 5700 50  0000 C CNN
 F 1 "220" V 1900 5700 50  0000 C CNN
 F 2 "Resistors_SMD:R_0603" V 1830 5700 50  0001 C CNN
@@
 $EndComp
 $Comp
-L R R5
+L R R8
 U 1 1 58F58F23
 P 1900 6000
-F 0 "R5" V 1980 6000 50  0000 C CNN
+F 0 "R8" V 1980 6000 50  0000 C CNN
 F 1 "220" V 1900 6000 50  0000 C CNN
 F 2 "Resistors_SMD:R_0603" V 1830 6000 50  0001 C CNN
@@
 $EndComp
 $Comp
-L R R10
+L R R13
 U 1 1 58F5A148
 P 1900 6300
-F 0 "R10" V 1980 6300 50  0000 C CNN
+F 0 "R13" V 1980 6300 50  0000 C CNN
 F 1 "220" V 1900 6300 50  0000 C CNN
 F 2 "Resistors_SMD:R_0603" V 1830 6300 50  0001 C CNN
@@
 $EndComp
 $Comp
-L R R6
+L R R9
 U 1 1 58F665D2
 P 1900 7500
-F 0 "R6" V 1980 7500 50  0000 C CNN
+F 0 "R9" V 1980 7500 50  0000 C CNN
 F 1 "220" V 1900 7500 50  0000 C CNN
 F 2 "Resistors_SMD:R_0603" V 1830 7500 50  0001 C CNN
@@
 $EndComp
 $Comp
-L R R11
+L R R14
 U 1 1 58F6D038
 P 2600 8500
-F 0 "R11" V 2680 8500 50  0000 C CNN
+F 0 "R14" V 2680 8500 50  0000 C CNN
 F 1 "27k" V 2600 8500 50  0000 C CNN
 F 2 "Resistors_SMD:R_0603" V 2530 8500 50  0001 C CNN
@@
 $EndComp
 $Comp
-L R R12
+L R R15
 U 1 1 58F6D79B
 P 2600 8900
-F 0 "R12" V 2680 8900 50  0000 C CNN
+F 0 "R15" V 2680 8900 50  0000 C CNN
 F 1 "47k" V 2600 8900 50  0000 C CNN
 F 2 "Resistors_SMD:R_0603" V 2530 8900 50  0001 C CNN
@@
 $EndComp
 $Comp
-L R R9
+L R R12
 U 1 1 58F715AE
 P 8300 8000
-F 0 "R9" V 8380 8000 50  0000 C CNN
+F 0 "R12" V 8380 8000 50  0000 C CNN
 F 1 "39" V 8300 8000 50  0000 C CNN
 F 2 "Resistors_SMD:R_0603" V 8230 8000 50  0001 C CNN
@@
 $EndComp
 $Comp
-L R R7
+L R R10
 U 1 1 58F716CE
 P 8800 8000
-F 0 "R7" V 8880 8000 50  0000 C CNN
+F 0 "R10" V 8880 8000 50  0000 C CNN
 F 1 "39" V 8800 8000 50  0000 C CNN
 F 2 "Resistors_SMD:R_0603" V 8730 8000 50  0001 C CNN
@@
 $EndComp
 $Comp
-L R R8
+L R R11
 U 1 1 58F71851
 P 8550 7750
-F 0 "R8" V 8630 7750 50  0000 C CNN
+F 0 "R11" V 8630 7750 50  0000 C CNN
 F 1 "100k" V 8550 7750 50  0000 C CNN
 F 2 "Resistors_SMD:R_0603" V 8480 7750 50  0001 C CNN
