File: NMEA_Multiplexer_v2.sch (KiCad schematic (older format))
At the start: 94 parts, among them J1 USB, J2 PoRt 1, J3 PoRt 2, J4 PoRt 3, J5 PoRt 4, J6 PoRt 5, J7 12V, J8 DEBUG UART, J9 JTAG, SW1 Reset, U1 ATSAMG55J19A-AU, U2 XR32330, U3 XR32330, U4 LF33ABDT-TR, U5 HM-11, Y1 32.768k

Commit message: Everything connected!
Connections:
- net labels added: CTS0, TCK
- net labels removed: CxTS0, TCxK
Changed lines of the file:
@@
 TMS
 Text Label 7550 10250 0    60   ~ 0
-TCxK
+TCK
 Text Label 7550 10350 0    60   ~ 0
 TDO
@@
 TMS
 Text Label 4900 2750 2    60   ~ 0
-TCxK
+TCK
 Text Label 4900 3900 2    60   ~ 0
 nRST
@@
 LED_0_ERR
 Text Label 9100 4350 0    60   ~ 0
-CxTS0
+CTS0
 Text Label 9100 2950 0    60   ~ 0
 LED_1_TX
@@
 TXD2
 Text Label 12350 5900 2    60   ~ 0
+RXD2
+Text Label 12350 6000 2    60   ~ 0
 RXD3
-Text Label 12350 6000 2    60   ~ 0
-RXD2
 Text Label 13750 5300 0    60   ~ 0
 TX3
@@
 TX4
 Text Label 13750 5900 0    60   ~ 0
+RX4
+Text Label 13750 6000 0    60   ~ 0
 RX3
-Text Label 13750 6000 0    60   ~ 0
-RX4
 NoConn ~ 13700 5500
 NoConn ~ 12400 6100
@@
 NoConn ~ 12350 7900
 Text Label 12250 7500 2    60   ~ 0
-CxTS0
+CTS0
 Text Label 12250 7600 2    60   ~ 0
 RXD0

Commit message: Updated USB footprint Connected BT KEY pin
Parts:
- D1: value Tx 3 (gReen) -> Tx 3 (green)
- D11: value Tx (gReen) -> Tx (green)
- D12: value ERr 2 (reD) -> Err 2 (red)
- D14: value Tx 1 (gReen) -> Tx 1 (green)
- D15: value ERr 1 (reD) -> Err 1 (red)
- D17: value Tx 0 (gReen) -> Tx 0 (green)
- D18: value ERr 0 (reD) -> Err 0 (red)
- D2: value ERr 3 (reD) -> Err 3 (red)
- D4: value Tx 4 (gReen) -> Tx 4 (green)
- D5: value ERr 4 (reD) -> Err 4 (red)
- D8: value BT Cxon (blue) -> BT Con (blue)
- D9: value Tx BT (gReen) -> Tx BT (green)
- J2: value PoRt 1 -> Port 1
- J3: value PoRt 2 -> Port 2
- J4: value PoRt 3 -> Port 3
- J5: value PoRt 4 -> Port 4
- J6: value PoRt 5 -> Port 5
Connections:
- net labels added: BT_KEY, LED_BT_CON
- net labels removed: LED_BT_CxON
- wire segments 331 -> 333
- no-connect marks 21 -> 19
Other:
- note added: "Close to\nVDDCORE"
- note added: "Close to\nVDDIO"
- note added: "Close to\nVDDOUT"
- note added: "Close to\nVDDUSB"
- note removed: "Cxlose to\nVDDCORE"
- note removed: "Cxlose to\nVDDIO"
- note removed: "Cxlose to\nVDDOUT"
- note removed: "Cxlose to\nVDDUSB"
Changed lines of the file:
@@
 $EndComp
 Text Notes 1200 11000 0    60   ~ 0
-Cxlose to\nVDDIO
+Close to\nVDDIO
 Text Notes 2300 11000 0    60   ~ 0
-Cxlose to\nVDDCORE
+Close to\nVDDCORE
 Text Notes 2900 11000 0    60   ~ 0
-Cxlose to\nVDDOUT
+Close to\nVDDOUT
 Text Notes 3500 11000 0    60   ~ 0
-Cxlose to\nVDDUSB
+Close to\nVDDUSB
 $Comp
 L Crystal_Small Y1
@@
 TXD2
 Text Label 4900 2050 2    60   ~ 0
+TXD6
+Text Label 4900 2150 2    60   ~ 0
 RXD6
-Text Label 4900 2150 2    60   ~ 0
-TXD6
 Text Label 9100 3050 0    60   ~ 0
 RXD5
@@
 P 1450 1350
 F 0 "D18" H 1450 1250 50  0000 C CNN
-F 1 "ERr 0 (reD)" H 1450 1450 50  0000 C CNN
+F 1 "Err 0 (red)" H 1450 1450 50  0000 C CNN
 F 2 "LEDs:LED_0603" H 1450 1350 50  0001 C CNN
 F 3 "" H 1450 1350 50  0001 C CNN
@@
 P 1450 1050
 F 0 "D17" H 1450 950 50  0000 C CNN
-F 1 "Tx 0 (gReen)" H 1450 1150 50  0000 C CNN
+F 1 "Tx 0 (green)" H 1450 1150 50  0000 C CNN
 F 2 "LEDs:LED_0603" H 1450 1050 50  0001 C CNN
 F 3 "" H 1450 1050 50  0001 C CNN
@@
 P 1450 2350
 F 0 "D15" H 1450 2250 50  0000 C CNN
-F 1 "ERr 1 (reD)" H 1450 2450 50  0000 C CNN
+F 1 "Err 1 (red)" H 1450 2450 50  0000 C CNN
 F 2 "LEDs:LED_0603" H 1450 2350 50  0001 C CNN
 F 3 "" H 1450 2350 50  0001 C CNN
@@
 P 1450 2050
 F 0 "D14" H 1450 1950 50  0000 C CNN
-F 1 "Tx 1 (gReen)" H 1450 2150 50  0000 C CNN
+F 1 "Tx 1 (green)" H 1450 2150 50  0000 C CNN
 F 2 "LEDs:LED_0603" H 1450 2050 50  0001 C CNN
 F 3 "" H 1450 2050 50  0001 C CNN
@@
 P 1450 3350
 F 0 "D12" H 1450 3250 50  0000 C CNN
-F 1 "ERr 2 (reD)" H 1450 3450 50  0000 C CNN
+F 1 "Err 2 (red)" H 1450 3450 50  0000 C CNN
 F 2 "LEDs:LED_0603" H 1450 3350 50  0001 C CNN
 F 3 "" H 1450 3350 50  0001 C CNN
@@
 P 1450 3050
 F 0 "D11" H 1450 2950 50  0000 C CNN
-F 1 "Tx (gReen)" H 1450 3150 50  0000 C CNN
+F 1 "Tx (green)" H 1450 3150 50  0000 C CNN
 F 2 "LEDs:LED_0603" H 1450 3050 50  0001 C CNN
 F 3 "" H 1450 3050 50  0001 C CNN
@@
 P 1450 4350
 F 0 "D2" H 1450 4250 50  0000 C CNN
-F 1 "ERr 3 (reD)" H 1450 4450 50  0000 C CNN
+F 1 "Err 3 (red)" H 1450 4450 50  0000 C CNN
 F 2 "LEDs:LED_0603" H 1450 4350 50  0001 C CNN
 F 3 "" H 1450 4350 50  0001 C CNN
@@
 P 1450 4050
 F 0 "D1" H 1450 3950 50  0000 C CNN
-F 1 "Tx 3 (gReen)" H 1450 4150 50  0000 C CNN
+F 1 "Tx 3 (green)" H 1450 4150 50  0000 C CNN
 F 2 "LEDs:LED_0603" H 1450 4050 50  0001 C CNN
 F 3 "" H 1450 4050 50  0001 C CNN
@@
 P 1450 5300
 F 0 "D5" H 1450 5200 50  0000 C CNN
-F 1 "ERr 4 (reD)" H 1450 5400 50  0000 C CNN
+F 1 "Err 4 (red)" H 1450 5400 50  0000 C CNN
 F 2 "LEDs:LED_0603" H 1450 5300 50  0001 C CNN
 F 3 "" H 1450 5300 50  0001 C CNN
@@
 P 1450 5000
 F 0 "D4" H 1450 4900 50  0000 C CNN
-F 1 "Tx 4 (gReen)" H 1450 5100 50  0000 C CNN
+F 1 "Tx 4 (green)" H 1450 5100 50  0000 C CNN
 F 2 "LEDs:LED_0603" H 1450 5000 50  0001 C CNN
 F 3 "" H 1450 5000 50  0001 C CNN
@@
 P 1450 6000
 F 0 "D9" H 1450 5900 50  0000 C CNN
-F 1 "Tx BT (gReen)" H 1450 6100 50  0000 C CNN
+F 1 "Tx BT (green)" H 1450 6100 50  0000 C CNN
 F 2 "LEDs:LED_0603" H 1450 6000 50  0001 C CNN
 F 3 "" H 1450 6000 50  0001 C CNN
@@
 P 1450 6300
 F 0 "D8" H 1450 6200 50  0000 C CNN
-F 1 "BT Cxon (blue)" H 1450 6400 50  0000 C CNN
+F 1 "BT Con (blue)" H 1450 6400 50  0000 C CNN
 F 2 "LEDs:LED_0603" H 1450 6300 50  0001 C CNN
 F 3 "" H 1450 6300 50  0001 C CNN
@@
 $EndComp
 Text Label 2150 6300 0    60   ~ 0
-LED_BT_CxON
+LED_BT_CON
 $Comp
 L CONN_01X03 J8
@@
 RXD6
 Text Label 13750 2250 0    60   ~ 0
-TX0
+TX2
 Text Label 13750 2350 0    60   ~ 0
 TX1
 Text Label 13750 2450 0    60   ~ 0
-TX2
+TX0
 Text Label 13750 2850 0    60   ~ 0
-RX0
+RX2
 Text Label 13750 2950 0    60   ~ 0
 RX1
 Text Label 13750 3050 0    60   ~ 0
-RX2
+RX0
 $Comp
 L XR32330 U2
@@
 P 3100 1100
 F 0 "J2" H 3100 1450 50  0000 C TNN
-F 1 "PoRt 1" V 2950 1100 50  0000 C TNN
+F 1 "Port 1" V 2950 1100 50  0000 C TNN
 F 2 "Connectors_Terminal_Blocks:TerminalBlock_Pheonix_PT-3.5mm_3pol" H 3100 775 50  0001 C CNN
 F 3 "" H 3075 1200 50  0001 C CNN
@@
 $EndComp
 Text Label 3550 900  0    60   ~ 0
-TX2
+TX0
 Text Label 3550 1300 0    60   ~ 0
-RX2
+RX0
 $Comp
 L GND #PWR042
@@
 P 3100 2100
 F 0 "J3" H 3100 2450 50  0000 C TNN
-F 1 "PoRt 2" V 2950 2100 50  0000 C TNN
+F 1 "Port 2" V 2950 2100 50  0000 C TNN
 F 2 "Connectors_Terminal_Blocks:TerminalBlock_Pheonix_PT-3.5mm_3pol" H 3100 1775 50  0001 C CNN
 F 3 "" H 3075 2200 50  0001 C CNN
@@
 P 3100 3100
 F 0 "J4" H 3100 3450 50  0000 C TNN
-F 1 "PoRt 3" V 2950 3100 50  0000 C TNN
+F 1 "Port 3" V 2950 3100 50  0000 C TNN
 F 2 "Connectors_Terminal_Blocks:TerminalBlock_Pheonix_PT-3.5mm_3pol" H 3100 2775 50  0001 C CNN
 F 3 "" H 3075 3200 50  0001 C CNN
@@
 $EndComp
 Text Label 3550 2900 0    60   ~ 0
-TX0
+TX2
 Text Label 3550 3300 0    60   ~ 0
-RX0
+RX2
 $Comp
 L GND #PWR044
@@
 P 3100 4100
 F 0 "J5" H 3100 4450 50  0000 C TNN
-F 1 "PoRt 4" V 2950 4100 50  0000 C TNN
+F 1 "Port 4" V 2950 4100 50  0000 C TNN
 F 2 "Connectors_Terminal_Blocks:TerminalBlock_Pheonix_PT-3.5mm_3pol" H 3100 3775 50  0001 C CNN
 F 3 "" H 3075 4200 50  0001 C CNN
@@
 P 3100 5100
 F 0 "J6" H 3100 5450 50  0000 C TNN
-F 1 "PoRt 5" V 2950 5100 50  0000 C TNN
+F 1 "Port 5" V 2950 5100 50  0000 C TNN
 F 2 "Connectors_Terminal_Blocks:TerminalBlock_Pheonix_PT-3.5mm_3pol" H 3100 4775 50  0001 C CNN
 F 3 "" H 3075 5200 50  0001 C CNN
@@
 NoConn ~ 13750 7700
 NoConn ~ 13750 7600
-NoConn ~ 13750 7900
 NoConn ~ 13750 8000
 NoConn ~ 13750 8100
@@
 TXD0
 Text Label 13850 7800 0    60   ~ 0
-LED_BT_CxON
+LED_BT_CON
 Text Label 13850 7500 0    60   ~ 0
 BT_RESET_N
@@
 Wire Wire Line
 	9100 3350 9000 3350
-NoConn ~ 9000 4150
 Wire Wire Line
 	9100 3450 9000 3450
@@
 	9100 4750 9000 4750
 Connection ~ 6900 1500
+Wire Wire Line
+	13850 7900 13750 7900
+Text Label 13850 7900 0    60   ~ 0
+BT_KEY
+Wire Wire Line
+	9100 4150 9000 4150
+Text Label 9100 4150 0    60   ~ 0
+BT_KEY
 $EndSCHEMATC
